Commit message: Update kr20.urdf

File: lab_ws/src/kuka_kr20_description/urdf/kr20.urdf (robot description, URDF)
Before this commit: robot kr20, 11 links, 10 joints
Links:
- removed link base
- removed link gripper
- removed link gripper_left
- removed link gripper_right
- removed link link01
- removed link link02
- removed link link03
- removed link link04
- removed link link05
- removed link link12
- added link link_00, mass 157.633; collision box size=0.3 0.3 1.3; visual box size=0.3 0.3 1.3
- added link link_01, mass 157.633; collision mesh filename=package://kuka_kr20_description/meshes/link01.stl scale=0.001 0.001 0.001; visual mesh filename=package://kuka_kr20_description/meshes/link01.stl scale=0.001 0.001 0.001
- added link link_02, mass 10; collision mesh filename=package://kuka_kr20_description/meshes/link02.stl scale=0.001 0.001 0.001; visual mesh filename=package://kuka_kr20_description/meshes/link02.stl scale=0.001 0.001 0.001
- added link link_03, mass 7; collision mesh filename=package://kuka_kr20_description/meshes/link03.stl scale=0.001 0.001 0.001; visual mesh filename=package://kuka_kr20_description/meshes/link03.stl scale=0.001 0.001 0.001
- added link link_04, mass 2; collision mesh filename=package://kuka_kr20_description/meshes/link04.stl scale=0.001 0.001 0.001; visual mesh filename=package://kuka_kr20_description/meshes/link04.stl scale=0.001 0.001 0.001
- added link link_05, mass 2; collision mesh filename=package://kuka_kr20_description/meshes/link05.stl scale=0.001 0.001 0.001; visual mesh filename=package://kuka_kr20_description/meshes/link05.stl scale=0.001 0.001 0.001
- added link link_12, mass 157.633; collision box size=0.6 0.3 0.3; visual box size=0.6 0.3 0.3
- added link pusher, mass 0.1; collision box size=0.02 0.18 0.1; visual box size=0.02 0.18 0.1
- added link shovel_base, mass 0.5; collision cylinder length=0.1 radius=0.05; visual cylinder length=0.1 radius=0.05
- added link shovel_plate, mass 0.2; collision box size=0.3 0.2 0.02; visual box size=0.3 0.2 0.02
Joints:
- removed joint base__link01
- removed joint gripper__gripper_left
- removed joint gripper__gripper_right
- removed joint link01__link02
- removed joint link02__link03
- removed joint link03__link04
- removed joint link04__link05
- removed joint link05__gripper
- removed joint link12__link01
- removed joint world__base
- added joint link05__shovel_base: type revolute, parent link_05, child shovel_base, origin xyz=0.115 0 0 rpy=0 0 0, axis 0 1 0, limit lower=-3.14 upper=3.14 effort=1000 velocity=0.5
- added joint link_00__link_12: type revolute, parent link_00, child link_12, origin xyz=0 0 0.15 rpy=0 0 0, axis 0 0 1, limit lower=-3.14 upper=3.14 effort=1000 velocity=0.5
- added joint link_01__link_02: type revolute, parent link_01, child link_02, origin xyz=0.160 -0.095 0.220 rpy=0 0 0, axis 0 1 0, limit lower=-1.5708 upper=1.7453 effort=1000 velocity=0.5
- added joint link_02__link_03: type revolute, parent link_02, child link_03, origin xyz=0.00 -0.01 0.780 rpy=0 0 0, axis 0 -1 0, limit lower=-1.55 upper=2 effort=1000 velocity=0.5
- added joint link_03__link_04: type revolute, parent link_03, child link_04, origin xyz=0.700 0.105 0.150 rpy=0 0 0, axis 1 0 0, limit lower=-3.0 upper=3.0 effort=1000 velocity=0.5
- added joint link_04__link_05: type revolute, parent link_04, child link_05, origin xyz=0.155 0.000 0.000 rpy=0 0 0, axis 0 -1 0, limit lower=-2.0 upper=2.0 effort=1000 velocity=0.5
- added joint link_12__link_01: type revolute, parent link_12, child link_01, origin xyz=0 0 0.15 rpy=0 0 0, axis 0 0 1, limit lower=-2 upper=2 effort=1000 velocity=0.5
- added joint shovel_base__pusher: type prismatic, parent shovel_base, child pusher, origin xyz=0.15 0 0 rpy=0 0 0, axis 1 0 0, limit lower=0 upper=0.25 effort=1000 velocity=0.5
- added joint shovel_base__shovel_plate: type fixed, parent shovel_base, child shovel_plate, origin xyz=0 0 0 rpy=0 0 0
- added joint world__link_00: type fixed, parent world, child link_00, origin xyz=0 0 0 rpy=0 0 0
